Commit message: 3-14

File: src/robotic_arm/urdf/robotic_arm.urdf (robot description, URDF)
Before this commit: robot robotic_arm, 8 links, 7 joints
Joints:
- joint joint4: limit lower=-3.14159 upper=3.14159 effort=50 velocity=10 -> lower=-3.926990716 upper=0.7853981633974483 effort=50 velocity=10

Commit message: urdf

File: src/robotic_arm/urdf/robotic_arm.urdf (robot description, URDF)
Before this commit: robot robotic_arm, 8 links, 7 joints
Joints:
- joint joint1: limit lower=-1.47 upper=1.47 effort=50 velocity=10 -> lower=-6.283185307 upper=6.283185307 effort=50 velocity=10
- joint joint2: limit lower=-1.134464014 upper=1.570796327 effort=50 velocity=10 -> lower=-1.570796327 upper=1.570796327 effort=50 velocity=10; origin xyz=0 0.03675 0.153 rpy=1.5708 -1.1579 0 -> xyz=0 0.03675 0.153 rpy=1.5708 -1.5708 0
- joint joint3: limit lower=0.0 upper=5.759586532 effort=50 velocity=10 -> lower=-3.141592654 upper=3.141592654 effort=50 velocity=10; origin xyz=0.52 0 0.08565 rpy=0 0 -2.7359 -> xyz=0.52 0 0.08565 rpy=0 0 0
- joint joint4: limit lower=-3.926990716 upper=0.7853981633974483 effort=50 velocity=10 -> lower=-3.141592654 upper=3.141592654 effort=50 velocity=10; origin xyz=0.436 0 0.0225 rpy=0 0 1.5836 -> xyz=0.436 0 0.0225 rpy=0 0 0
- joint joint6: origin xyz=0.073796 0.0036822 8.8922E-05 rpy=0.051163 -1.5708 0 -> xyz=0.073796 0.0036822 8.8922E-05 rpy=0 -1.5708 0
